Commit message: fix the color model error.

File: scripts/robots/GIRONA500ARM5.urdf (robot description, URDF)
Before this commit: robot girona500, 10 links, 9 joints
Links:
- link base_link: geometry visual mesh filename=GIRONA500/g500_March11.osg
- link part0: geometry visual mesh filename=ARM5E/ARM5E_part0.osg
- link part1: geometry visual mesh filename=ARM5E/ARM5E_part1.osg
- link part2: geometry visual mesh filename=ARM5E/ARM5E_part2.osg
- link part3: geometry visual mesh filename=ARM5E/ARM5E_part3.osg
- link part4_base: geometry visual mesh filename=ARM5E/ARM5E_part4_base.osg
- link part4_jaw1: geometry visual mesh filename=ARM5E/ARM5E_part4_jaw1.osg
- link part4_jaw2: geometry visual mesh filename=ARM5E/ARM5E_part4_jaw2.osg
